Commit message: v-5 updated single point and multi point models for hardware targets, added mask-r-cnn codes for target detection without its model

File: urdf/urdf/lite6.urdf (robot description, URDF)
Before this commit: robot UF_ROBOT, 9 links, 8 joints
Joints:
- joint joint2: origin xyz=0 0 0 rpy=1.5708 -0.7854 3.1416 -> xyz=0 0 0 rpy=1.5708 -2.0315632493 3.1416
- joint joint3: origin xyz=0.2002 0 0 rpy=-3.1416 0 0.7854 -> xyz=0.2002 0 0 rpy=-3.1416 0 -0.4694935688
- joint joint4: origin xyz=0.087 -0.22761 0 rpy=1.5708 0 0 -> xyz=0.087 -0.22761 0 rpy=1.5708 -0.0174532925 0
- joint joint5: origin xyz=0 0 0 rpy=1.5708 -1.5708 0 -> xyz=0 0 0 rpy=1.5708 -1.4573499254 0

Commit message: v-8 updated to multi target point and trained with certain bounding box

File: urdf/urdf/lite6.urdf (robot description, URDF)
Before this commit: robot UF_ROBOT, 9 links, 8 joints
Joints:
- joint joint2: origin xyz=0 0 0 rpy=1.5708 -2.0315632493 3.1416 -> xyz=0 0 0 rpy=1.5708 -0.7854 3.1416
- joint joint3: origin xyz=0.2002 0 0 rpy=-3.1416 0 -0.4694935688 -> xyz=0.2002 0 0 rpy=-3.1416 0 0.7854
- joint joint4: origin xyz=0.087 -0.22761 0 rpy=1.5708 -0.0174532925 0 -> xyz=0.087 -0.22761 0 rpy=1.5708 0 0
- joint joint5: origin xyz=0 0 0 rpy=1.5708 -1.4573499254 0 -> xyz=0 0 0 rpy=1.5708 -1.5708 0
